File: EEG2.sch (KiCad schematic (older format))
At the start: 102 parts, among them J1Input1 Conn_Coaxial, J2Input2 Conn_Coaxial, J3InputGround1 Conn_Coaxial

Commit message: dan cant github
Parts:
- removed PWRGroundZoneConnect1: 0, Resistor_THT:R_Axial_DIN0207_L6.3mm_D2.5mm_P10.16mm_Horizontal, symbol Device:R_Small_US
- added CaseGND1: ., Resistor_THT:R_Axial_DIN0207_L6.3mm_D2.5mm_P10.16mm_Horizontal, symbol Device:R_Small_US
- BNCOut1: renamed from BNC_OUT1; value Conn_Coaxial -> BNCOut
- J1In1: renamed from J1Input1; value Conn_Coaxial -> BNCIn1
- J2In2: renamed from J2Input2; value Conn_Coaxial -> BNCIn2
- J3InGND1: renamed from J3InputGround1; value Conn_Coaxial -> BNCGnd
- KK_KF2510: value Conn_01x03_Male -> KK_KF2510
- PinOut1: renamed from PIN_OUT1; value Conn_01x02_Male -> 01x02Male
- SCoup2: renamed from SupplyCoupling2; footprint Capacitor_SMD:C_Elec_4x5.4 -> Capacitor_THT:C_Radial_D10.0mm_H12.5mm_P5.00mm
- SCoup4: renamed from SupplyCoupling4; footprint Capacitor_SMD:C_Elec_4x5.4 -> Capacitor_THT:C_Radial_D10.0mm_H12.5mm_P5.00mm
- renumbered ACoupling1 to ACoup1, ACoupling2 to ACoup2, BConnect1 to BCon1, BConnect2 to BCon2, BCoupling1 to BCoup1, BCoupling2 to BCoup2, BGroundConnect1 to BGNDCon1, CConnect1 to CCon1, DConnect1 to DCon1, DCoupling1 to DCoup1, DCoupling2 to DCoup2, DCoupling3 to DCoup3, DCoupling4 to DCoup4, EConnect1 to ECon1, ECoupling1 to ECoup1, ECoupling2 to ECoup2, ECoupling3 to ECoup3, ECoupling4 to ECoup4, FConnect1 to FCon1, FCoupling1 to FCoup1, FCoupling2 to FCoup2, FCoupling3 to FCoup3, FCoupling4 to FCoup4, GConnect1 to GCon1, GCoupling1 to GCoup1, GCoupling2 to GCoup2, HConnect1 to HCon1, HCoupling1 to HCoup1, HCoupling2 to HCoup2, HCoupling3 to HCoup3, HCoupling4 to HCoup4, IConnect1 to ICon1, ICoupling1 to ICoup1, ICoupling2 to ICoup2, POWER_SUPPLY_P1G2N3 to POW_1+2G3-1, SupplyCoupling1 to SCoup1, SupplyCoupling3 to SCoup3
Connections:
- net GND: now also CaseGND1.1, CaseGND1.2
